Commit message: pre-commit fmt

File: urdf/materials.xacro (robot description, xacro)
@@ -1,3 +1,3 @@
-<?xml version="1.0" ?>
+<?xml version="1.0"?>
 <robot name="xacro_properties" xmlns:xacro="http://ros.org/wiki/xacro">
   <material name="Grey">

File: urdf/robotiq_hande_gripper.ros2_control.xacro (robot description, xacro)
@@ -1,27 +1,27 @@
 <?xml version="1.0"?>
 <robot xmlns:xacro="http://www.ros.org/wiki/xacro">
-    <xacro:macro name="robotiq_hande_ros2_control" params="name prefix tty use_fake_hardware:=false">
-        <ros2_control name="${name}" type="system">
-          <hardware>
-            <xacro:if value="${use_fake_hardware}">
-                  <plugin>mock_components/GenericSystem</plugin>
-            </xacro:if>
-            <xacro:unless value="${use_fake_hardware}">
-              <plugin>robotiq_hande_driver/RobotiqHandeHardwareInterface</plugin>
-              <param name="tty">${tty}</param>
-            </xacro:unless>
-          </hardware>
-            <!-- The right finger joint uses the mimic feature -->
-            <joint name="${prefix}hande_left_finger_joint">
-              <command_interface name="position">
-                <param name="min">0</param>
-                <param name="max">0.025</param>
-              </command_interface>
-              <state_interface name="position">
-                  <param name="initial_value">0.025</param>
-              </state_interface>
-              <state_interface name="velocity"/>
-            </joint>
-        </ros2_control>
-    </xacro:macro>
+  <xacro:macro name="robotiq_hande_ros2_control" params="name prefix tty use_fake_hardware:=false">
+    <ros2_control name="${name}" type="system">
+      <hardware>
+        <xacro:if value="${use_fake_hardware}">
+          <plugin>mock_components/GenericSystem</plugin>
+        </xacro:if>
+        <xacro:unless value="${use_fake_hardware}">
+          <plugin>robotiq_hande_driver/RobotiqHandeHardwareInterface</plugin>
+          <param name="tty">${tty}</param>
+        </xacro:unless>
+      </hardware>
+      <!-- The right finger joint uses the mimic feature -->
+      <joint name="${prefix}hande_left_finger_joint">
+        <command_interface name="position">
+          <param name="min">0</param>
+          <param name="max">0.025</param>
+        </command_interface>
+        <state_interface name="position">
+          <param name="initial_value">0.025</param>
+        </state_interface>
+        <state_interface name="velocity"/>
+      </joint>
+    </ros2_control>
+  </xacro:macro>
 </robot>

File: urdf/robotiq_hande_gripper.urdf.xacro (robot description, xacro)
@@ -1,10 +1,9 @@
 <?xml version="1.0"?>
-<robot xmlns:xacro="http://ros.org/wiki/xacro"
-       name="robotiq_hande_gripper" >
-  <xacro:arg name="parent" default="tool0" />
-  <xacro:arg name="tty" default="/dev/ttyXXX" />
-  <xacro:arg name="use_fake_hardware" default="true" />
-  <xacro:include filename="$(find robotiq_hande_description)/urdf/robotiq_hande_gripper.xacro" />
-  <link name="$(arg parent)" />
-  <xacro:robotiq_hande_gripper name="robotiq_hande_gripper" prefix="" parent="$(arg parent)" tty="$(arg tty)" use_fake_hardware="$(arg use_fake_hardware)" />
+<robot xmlns:xacro="http://ros.org/wiki/xacro" name="robotiq_hande_gripper">
+  <xacro:arg name="parent" default="tool0"/>
+  <xacro:arg name="tty" default="/dev/ttyXXX"/>
+  <xacro:arg name="use_fake_hardware" default="true"/>
+  <xacro:include filename="$(find robotiq_hande_description)/urdf/robotiq_hande_gripper.xacro"/>
+  <link name="$(arg parent)"/>
+  <xacro:robotiq_hande_gripper name="robotiq_hande_gripper" prefix="" parent="$(arg parent)" tty="$(arg tty)" use_fake_hardware="$(arg use_fake_hardware)"/>
 </robot>

File: urdf/robotiq_hande_gripper.xacro (robot description, xacro)
@@ -4,18 +4,14 @@
     Based on the URDF file by Cristian C Beltran-Hernandez
   -->
-  <xacro:include filename="$(find robotiq_hande_description)/urdf/materials.xacro" />
-  <xacro:include filename="$(find robotiq_hande_description)/urdf/robotiq_hande_gripper.ros2_control.xacro" />
+  <xacro:include filename="$(find robotiq_hande_description)/urdf/materials.xacro"/>
+  <xacro:include filename="$(find robotiq_hande_description)/urdf/robotiq_hande_gripper.ros2_control.xacro"/>
   <xacro:macro name="robotiq_hande_gripper" params="name prefix parent tty use_fake_hardware">
     <!-- ros2_control parameters  -->
-    <xacro:robotiq_hande_ros2_control
-        name="${name}"
-        prefix="${prefix}"
-        tty="${tty}"
-        use_fake_hardware="${use_fake_hardware}" />
+    <xacro:robotiq_hande_ros2_control name="${name}" prefix="${prefix}" tty="${tty}" use_fake_hardware="${use_fake_hardware}"/>
     <!-- Robotiq Coupler -->
     <!--  + Height added by the coupler: 13.9mm -->
     <!--  + Reference frame: at the middle (6.95mm) -->
     <joint name="robotiq_hande_coupler_joint" type="fixed">
-      <origin xyz="0 0 0.00695" rpy="0 0 ${-pi/2.0}" />
+      <origin xyz="0 0 0.00695" rpy="0 0 ${-pi/2.0}"/>
       <parent link="${parent}"/>
       <child link="${prefix}robotiq_hande_coupler"/>
@@ -23,10 +19,6 @@
     <link name="${prefix}robotiq_hande_coupler">
       <inertial>
-        <mass value="0.168" />
-        <inertia
-          ixx="6.17674E-05" ixy="0.0" ixz="0.0"
-          iyy="6.17674E-05" iyz="0.0"
-          izz="1.18125E-04"
-        />
+        <mass value="0.168"/>
+        <inertia ixx="6.17674E-05" ixy="0.0" ixz="0.0" iyy="6.17674E-05" iyz="0.0" izz="1.18125E-04"/>
       </inertial>
       <collision>
@@ -37,7 +29,7 @@
       <visual>
         <geometry>
-          <mesh filename="package://robotiq_hande_description/meshes/coupler.dae" />
+          <mesh filename="package://robotiq_hande_description/meshes/coupler.dae"/>
         </geometry>
-        <material name="DarkGrey" />
+        <material name="DarkGrey"/>
       </visual>
     </link>
@@ -50,9 +42,5 @@
       <inertial>
         <mass value="0.86387"/>
-        <inertia
-          ixx="0.001" ixy="0.0" ixz="0.0"
-          iyy="0.001" iyz="0.0"
-          izz="0.0006"
-        />
+        <inertia ixx="0.001" ixy="0.0" ixz="0.0" iyy="0.001" iyz="0.0" izz="0.0006"/>
       </inertial>
       <collision>
@@ -80,9 +68,5 @@
         <origin rpy="0 0 0" xyz="0 0 0"/>
         <mass value="0.03804"/>
-        <inertia
-          ixx="1E-9" ixy="0.0" ixz="0.0"
-          iyy="1E-9" iyz="0.0"
-          izz="1E-9"
-        />
+        <inertia ixx="1E-9" ixy="0.0" ixz="0.0" iyy="1E-9" iyz="0.0" izz="1E-9"/>
       </inertial>
       <collision>
@@ -112,9 +96,5 @@
         <origin rpy="0 0 0" xyz="0 0 0"/>
         <mass value="0.03804"/>
-        <inertia
-          ixx="1E-9" ixy="0.0" ixz="0.0"
-          iyy="1E-9" iyz="0.0"
-          izz="1E-9"
-        />
+        <inertia ixx="1E-9" ixy="0.0" ixz="0.0" iyy="1E-9" iyz="0.0" izz="1E-9"/>
       </inertial>
       <collision>
@@ -129,5 +109,5 @@
           <mesh filename="package://robotiq_hande_description/meshes/finger.dae" scale="1.0 1.0 1.0"/>
         </geometry>
-        <material name="Grey" />
+        <material name="Grey"/>
       </visual>
     </link>
@@ -137,5 +117,5 @@
       <child link="${prefix}robotiq_hande_end"/>
     </joint>
-    <link name="${prefix}robotiq_hande_end" />
+    <link name="${prefix}robotiq_hande_end"/>
   </xacro:macro>
 </robot>
