Commit message: minor typos

File: urdf/robotiq_hande_gripper.ros2_control.xacro (robot description, xacro)
@@ -13,5 +13,5 @@
       </hardware>
       <!-- The right finger joint uses the mimic feature -->
-      <joint name="${prefix}hande_left_finger_joint">
+      <joint name="${prefix}robotiq_hande_left_finger_joint">
         <command_interface name="position">
           <param name="min">0</param>

File: urdf/robotiq_hande_gripper.xacro (robot description, xacro)
@@ -10,6 +10,6 @@
     <xacro:robotiq_hande_ros2_control name="${name}" prefix="${prefix}" tty="${tty}" use_fake_hardware="${use_fake_hardware}"/>
     <!-- Robotiq Coupler -->
-    <!--  + Height added by the coupler: 13.9mm -->
-    <!--  + Reference frame: at the middle (6.95mm) -->
+    <!--  + Height added by the coupler (13.9mm) -->
+    <!--  + Reference frame at the middle (6.95mm) -->
     <joint name="robotiq_hande_coupler_joint" type="fixed">
       <origin xyz="0 0 0.00695" rpy="0 0 ${-pi/2.0}"/>

Commit message: ADD: connection params

File: urdf/robotiq_hande_gripper.ros2_control.xacro (robot description, xacro)
@@ -1,5 +1,5 @@
 <?xml version="1.0"?>
 <robot xmlns:xacro="http://www.ros.org/wiki/xacro">
-  <xacro:macro name="robotiq_hande_ros2_control" params="name prefix tty use_fake_hardware:=false">
+  <xacro:macro name="robotiq_hande_ros2_control" params="name prefix grip_pos_min grip_pos_max tty baudrate parity data_bits stop_bit slave_id use_fake_hardware:=false">
     <ros2_control name="${name}" type="system">
       <hardware>
@@ -9,5 +9,12 @@
         <xacro:unless value="${use_fake_hardware}">
           <plugin>robotiq_hande_driver/RobotiqHandeHardwareInterface</plugin>
+          <param name="grip_pos_min">${grip_pos_min}</param>
+          <param name="grip_pos_max">${grip_pos_max}</param>
           <param name="tty">${tty}</param>
+          <param name="baudrate">${baudrate}</param>
+          <param name="parity">${parity}</param>
+          <param name="data_bits">${data_bits}</param>
+          <param name="stop_bit">${stop_bit}</param>
+          <param name="slave_id">${slave_id}</param>
         </xacro:unless>
       </hardware>

File: urdf/robotiq_hande_gripper.xacro (robot description, xacro)
@@ -6,7 +6,7 @@
   <xacro:include filename="$(find robotiq_hande_description)/urdf/materials.xacro"/>
   <xacro:include filename="$(find robotiq_hande_description)/urdf/robotiq_hande_gripper.ros2_control.xacro"/>
-  <xacro:macro name="robotiq_hande_gripper" params="name prefix parent tty use_fake_hardware">
+  <xacro:macro name="robotiq_hande_gripper" params="name prefix parent grip_pos_min grip_pos_max tty baudrate parity data_bits stop_bit slave_id use_fake_hardware">
     <!-- ros2_control parameters  -->
-    <xacro:robotiq_hande_ros2_control name="${name}" prefix="${prefix}" tty="${tty}" use_fake_hardware="${use_fake_hardware}"/>
+    <xacro:robotiq_hande_ros2_control name="${name}" prefix="${prefix}" grip_pos_min="${grip_pos_min}" grip_pos_max="${grip_pos_max}" tty="${tty}" baudrate="${baudrate}" parity="${parity}" data_bits="${data_bits}" stop_bit="${stop_bit}" slave_id="${slave_id}" use_fake_hardware="${use_fake_hardware}"/>
     <!-- Robotiq Coupler -->
     <!--  + Height added by the coupler (13.9mm) -->

Commit message: Configuration params for ModbusRTU serial communication (#1)
* ADD: connection params

* ADD: parameter config

* FIX: formatting

* FIX: initial velocity state value

* FIX: tty string

* CHG: put params in conditional statement

* FIX: formatting xacro

* ADD: changelog

File: urdf/robotiq_hande_gripper.ros2_control.xacro (robot description, xacro)
@@ -1,5 +1,5 @@
 <?xml version="1.0"?>
 <robot xmlns:xacro="http://www.ros.org/wiki/xacro">
-  <xacro:macro name="robotiq_hande_ros2_control" params="name prefix tty use_fake_hardware:=false">
+  <xacro:macro name="robotiq_hande_ros2_control" params="name prefix grip_pos_min grip_pos_max tty baudrate parity data_bits stop_bit slave_id use_fake_hardware:=false">
     <ros2_control name="${name}" type="system">
       <hardware>
@@ -9,5 +9,12 @@
         <xacro:unless value="${use_fake_hardware}">
           <plugin>robotiq_hande_driver/RobotiqHandeHardwareInterface</plugin>
-          <param name="tty">${tty}</param>
+          <param name="grip_pos_min">"${grip_pos_min}"</param>
+          <param name="grip_pos_max">"${grip_pos_max}"</param>
+          <param name="tty">"${tty}"</param>
+          <param name="baudrate">"${baudrate}"</param>
+          <param name="parity">"${parity}"</param>
+          <param name="data_bits">"${data_bits}"</param>
+          <param name="stop_bit">"${stop_bit}"</param>
+          <param name="slave_id">"${slave_id}"</param>
         </xacro:unless>
       </hardware>
@@ -21,5 +28,7 @@
           <param name="initial_value">0.025</param>
         </state_interface>
-        <state_interface name="velocity"/>
+        <state_interface name="velocity">
+          <param name="initial_value">0</param>
+        </state_interface>
       </joint>
     </ros2_control>

File: urdf/robotiq_hande_gripper.urdf.xacro (robot description, xacro)
@@ -2,8 +2,28 @@
 <robot xmlns:xacro="http://ros.org/wiki/xacro" name="robotiq_hande_gripper">
   <xacro:arg name="parent" default="tool0"/>
-  <xacro:arg name="tty" default="/dev/ttyXXX"/>
+  <xacro:arg name="grip_pos_min" default="0"/>
+  <xacro:arg name="grip_pos_max" default="0.025"/>
+  <xacro:arg name="tty" default="/tmp/ttyUR"/>
+  <xacro:arg name="baudrate" default="115200"/>
+  <xacro:arg name="parity" default="N"/>
+  <xacro:arg name="data_bits" default="8"/>
+  <xacro:arg name="stop_bit" default="1"/>
+  <xacro:arg name="slave_id" default="9"/>
   <xacro:arg name="use_fake_hardware" default="true"/>
   <xacro:include filename="$(find robotiq_hande_description)/urdf/robotiq_hande_gripper.xacro"/>
   <link name="$(arg parent)"/>
-  <xacro:robotiq_hande_gripper name="robotiq_hande_gripper" prefix="" parent="$(arg parent)" tty="$(arg tty)" use_fake_hardware="$(arg use_fake_hardware)"/>
+  <xacro:robotiq_hande_gripper
+    name="robotiq_hande_gripper"
+    prefix=""
+    parent="$(arg parent)"
+    grip_pos_min="$(arg grip_pos_min)"
+    grip_pos_max="$(arg grip_pos_max)"
+    tty="$(arg tty)"
+    baudrate="$(arg baudrate)"
+    parity="$(arg parity)"
+    data_bits="$(arg data_bits)"
+    stop_bit="$(arg stop_bit)"
+    slave_id="$(arg slave_id)"
+    use_fake_hardware="$(use_fake_hardware)"
+  />
 </robot>

File: urdf/robotiq_hande_gripper.xacro (robot description, xacro)
@@ -6,7 +6,19 @@
   <xacro:include filename="$(find robotiq_hande_description)/urdf/materials.xacro"/>
   <xacro:include filename="$(find robotiq_hande_description)/urdf/robotiq_hande_gripper.ros2_control.xacro"/>
-  <xacro:macro name="robotiq_hande_gripper" params="name prefix parent tty use_fake_hardware">
+  <xacro:macro name="robotiq_hande_gripper" params="name prefix parent grip_pos_min grip_pos_max tty baudrate parity data_bits stop_bit slave_id use_fake_hardware">
     <!-- ros2_control parameters  -->
-    <xacro:robotiq_hande_ros2_control name="${name}" prefix="${prefix}" tty="${tty}" use_fake_hardware="${use_fake_hardware}"/>
+    <xacro:robotiq_hande_ros2_control
+      name="${name}"
+      prefix="${prefix}"
+      grip_pos_min="${grip_pos_min}"
+      grip_pos_max="${grip_pos_max}"
+      tty="${tty}"
+      baudrate="${baudrate}"
+      parity="${parity}"
+      data_bits="${data_bits}"
+      stop_bit="${stop_bit}"
+      slave_id="${slave_id}"
+      use_fake_hardware="${use_fake_hardware}"
+    />
     <!-- Robotiq Coupler -->
     <!--  + Height added by the coupler (13.9mm) -->

Commit message: update ros2_control args

File: urdf/robotiq_hande_gripper.ros2_control.xacro (robot description, xacro)
@@ -1,5 +1,5 @@
 <?xml version="1.0"?>
 <robot xmlns:xacro="http://www.ros.org/wiki/xacro">
-  <xacro:macro name="robotiq_hande_ros2_control" params="name prefix tty use_fake_hardware:=false">
+  <xacro:macro name="robotiq_hande_ros2_control" params="name prefix tty use_fake_hardware">
     <ros2_control name="${name}" type="system">
       <hardware>
