Commit message: initial ros2_control params

File: urdf/robotiq_hande_gripper.urdf.xacro (robot description, xacro)
@@ -2,6 +2,9 @@
 <robot xmlns:xacro="http://ros.org/wiki/xacro"
        name="robotiq_hande_gripper" >
+  <xacro:arg name="parent" default="tool0" />
+  <xacro:arg name="tty" default="/dev/ttyXXX" />
+  <xacro:arg name="use_fake_hardware" default="true" />
   <xacro:include filename="$(find robotiq_hande_description)/urdf/robotiq_hande_gripper.xacro" />
-  <link name="tool0" />
-  <xacro:robotiq_hande_gripper parent="tool0" prefix="" />
+  <link name="$(arg parent)" />
+  <xacro:robotiq_hande_gripper name="robotiq_hande_gripper" prefix="" parent="$(arg parent)" tty="$(arg tty)" use_fake_hardware="$(arg use_fake_hardware)" />
 </robot>

File: urdf/robotiq_hande_gripper.xacro (robot description, xacro)
@@ -5,5 +5,12 @@
   -->
   <xacro:include filename="$(find robotiq_hande_description)/urdf/materials.xacro" />
-  <xacro:macro name="robotiq_hande_gripper" params="prefix parent">
+  <xacro:include filename="$(find robotiq_hande_description)/urdf/robotiq_hande_gripper.ros2_control.xacro" />
+  <xacro:macro name="robotiq_hande_gripper" params="name prefix parent tty use_fake_hardware">
+    <!-- ros2_control parameters  -->
+    <xacro:robotiq_hande_ros2_control
+        name="${name}"
+        prefix="${prefix}"
+        tty="${tty}"
+        use_fake_hardware="${use_fake_hardware}" />
     <!-- Robotiq Coupler -->
     <!--  + Height added by the coupler: 13.9mm -->

Commit message: pre-commit fmt

File: urdf/robotiq_hande_gripper.urdf.xacro (robot description, xacro)
@@ -1,7 +1,6 @@
 <?xml version="1.0"?>
-<robot xmlns:xacro="http://ros.org/wiki/xacro"
-       name="robotiq_hande_gripper" >
-  <xacro:include filename="$(find robotiq_hande_description)/urdf/robotiq_hande_gripper.xacro" />
-  <link name="tool0" />
-  <xacro:robotiq_hande_gripper parent="tool0" prefix="" />
+<robot xmlns:xacro="http://ros.org/wiki/xacro" name="robotiq_hande_gripper">
+  <xacro:include filename="$(find robotiq_hande_description)/urdf/robotiq_hande_gripper.xacro"/>
+  <link name="tool0"/>
+  <xacro:robotiq_hande_gripper parent="tool0" prefix=""/>
 </robot>

File: urdf/robotiq_hande_gripper.xacro (robot description, xacro)
@@ -4,5 +4,5 @@
     Based on the URDF file by Cristian C Beltran-Hernandez
   -->
-  <xacro:include filename="$(find robotiq_hande_description)/urdf/materials.xacro" />
+  <xacro:include filename="$(find robotiq_hande_description)/urdf/materials.xacro"/>
   <xacro:macro name="robotiq_hande_gripper" params="prefix parent">
     <!-- Robotiq Coupler -->
@@ -10,5 +10,5 @@
     <!--  + Reference frame: at the middle (6.95mm) -->
     <joint name="robotiq_coupler_joint" type="fixed">
-      <origin xyz="0 0 0.00695" rpy="0 0 ${-pi/2.0}" />
+      <origin xyz="0 0 0.00695" rpy="0 0 ${-pi/2.0}"/>
       <parent link="${parent}"/>
       <child link="${prefix}robotiq_coupler"/>
@@ -16,10 +16,6 @@
     <link name="${prefix}robotiq_coupler">
       <inertial>
-        <mass value="0.168" />
-        <inertia
-          ixx="6.17674E-05" ixy="0.0" ixz="0.0"
-          iyy="6.17674E-05" iyz="0.0"
-          izz="1.18125E-04"
-        />
+        <mass value="0.168"/>
+        <inertia ixx="6.17674E-05" ixy="0.0" ixz="0.0" iyy="6.17674E-05" iyz="0.0" izz="1.18125E-04"/>
       </inertial>
       <collision>
@@ -30,7 +26,7 @@
       <visual>
         <geometry>
-          <mesh filename="package://robotiq_hande_description/meshes/coupler.dae" />
+          <mesh filename="package://robotiq_hande_description/meshes/coupler.dae"/>
         </geometry>
-        <material name="DarkGrey" />
+        <material name="DarkGrey"/>
       </visual>
     </link>
@@ -43,9 +39,5 @@
       <inertial>
         <mass value="0.86387"/>
-        <inertia
-          ixx="0.001" ixy="0.0" ixz="0.0"
-          iyy="0.001" iyz="0.0"
-          izz="0.0006"
-        />
+        <inertia ixx="0.001" ixy="0.0" ixz="0.0" iyy="0.001" iyz="0.0" izz="0.0006"/>
       </inertial>
       <collision>
@@ -73,9 +65,5 @@
         <origin rpy="0 0 0" xyz="0 0 0"/>
         <mass value="0.03804"/>
-        <inertia
-          ixx="1E-9" ixy="0.0" ixz="0.0"
-          iyy="1E-9" iyz="0.0"
-          izz="1E-9"
-        />
+        <inertia ixx="1E-9" ixy="0.0" ixz="0.0" iyy="1E-9" iyz="0.0" izz="1E-9"/>
       </inertial>
       <collision>
@@ -105,9 +93,5 @@
         <origin rpy="0 0 0" xyz="0 0 0"/>
         <mass value="0.03804"/>
-        <inertia
-          ixx="1E-9" ixy="0.0" ixz="0.0"
-          iyy="1E-9" iyz="0.0"
-          izz="1E-9"
-        />
+        <inertia ixx="1E-9" ixy="0.0" ixz="0.0" iyy="1E-9" iyz="0.0" izz="1E-9"/>
       </inertial>
       <collision>
@@ -122,5 +106,5 @@
           <mesh filename="package://robotiq_hande_description/meshes/finger.dae" scale="1.0 1.0 1.0"/>
         </geometry>
-        <material name="Grey" />
+        <material name="Grey"/>
       </visual>
     </link>
@@ -130,5 +114,5 @@
       <child link="${prefix}hande_end"/>
     </joint>
-    <link name="${prefix}hande_end" />
+    <link name="${prefix}hande_end"/>
   </xacro:macro>
 </robot>

Commit message: redefined meshes and updated FCstd files

File: urdf/robotiq_hande_gripper.urdf.xacro (robot description, xacro)
@@ -25,5 +25,5 @@
     stop_bit="$(arg stop_bit)"
     slave_id="$(arg slave_id)"
-    use_fake_hardware="$(use_fake_hardware)"
+    use_fake_hardware="$(arg use_fake_hardware)"
   />
 </robot>

File: urdf/robotiq_hande_gripper.xacro (robot description, xacro)
@@ -20,13 +20,15 @@
       use_fake_hardware="${use_fake_hardware}"
     />
-    <!-- Robotiq Coupler -->
-    <!--  + Height added by the coupler (16.9mm) -->
-    <!--  + Reference frame at the middle (6.95mm) -->
+    <!-- Robotiq Hand-E specs -->
+    <!--  + Height added by the IO coupler: 11.0mm -->
+    <!--  + Height added by the Hand-E: 99.0mm -->
     <!--  + Coupler mass includes the bolts -->
-    <xacro:arg name="base_joint_z_offset" default="0.055"/>
-    <xacro:arg name="coupler_depth" default="0.00294"/>
-    <xacro:arg name="base_to_coupler_offset" default="0.00145"/>
+    <xacro:arg name="coupler_height" default="0.011"/>
+    <xacro:arg name="coupler_shell_height" default="0.0169"/>
+    <xacro:arg name="coupler_parent_cutoff" default="0.003"/>
+    <xacro:arg name="coupler_hande_cutoff" default="0.0029"/>
+    <xacro:arg name="hande_height" default="0.099"/>
     <joint name="${prefix}robotiq_hande_coupler_joint" type="fixed">
-      <origin xyz="0 0 0.00695" rpy="0 0 ${-pi/2.0}"/>
+      <origin xyz="0 0 0" rpy="0 0 ${-pi/2.0}"/>
       <parent link="${parent}"/>
       <child link="${prefix}robotiq_hande_coupler"/>
@@ -39,15 +41,17 @@
       </visual>
       <collision>
+        <origin xyz="0 0 ${$(arg coupler_shell_height)/2 - $(arg coupler_parent_cutoff)}" rpy="0 0 0"/>
         <geometry>
-          <cylinder length="0.014" radius="0.039"/>
+          <cylinder length="$(arg coupler_shell_height)" radius="0.039"/>
         </geometry>
       </collision>
       <inertial>
         <mass value="${coupler_mass}"/>
+        <!-- TODO: Parametrize intertia in terms of perpendicular axis to a solid cylinder -->
         <inertia ixx="6.17674E-5" ixy="0.0" ixz="0.0" iyy="6.17674E-5" iyz="0.0" izz="1.18125E-4"/>
       </inertial>
     </link>
     <joint name="${prefix}robotiq_hande_base_joint" type="fixed">
-      <origin xyz="0 0 ${$(arg base_joint_z_offset) + $(arg coupler_depth) - $(arg base_to_coupler_offset)}" rpy="0 0 0"/>
+      <origin xyz="0 0 $(arg coupler_height)" rpy="0 0 0"/>
       <parent link="${prefix}robotiq_hande_coupler"/>
       <child link="${prefix}robotiq_hande_link"/>
@@ -55,5 +59,5 @@
     <link name="${prefix}robotiq_hande_link">
       <visual>
-        <origin xyz="0 0 0" rpy="0 ${-pi/2} 0"/>
+        <origin xyz="0 0 0" rpy="0 0 0"/>
         <geometry>
           <mesh filename="package://robotiq_hande_description/meshes/hande.dae" scale="1.0 1.0 1.0"/>
@@ -61,15 +65,17 @@
       </visual>
       <collision>
+        <origin xyz="0 0 ${($(arg hande_height) + $(arg coupler_hande_cutoff) + 0.005) / 2}" rpy="0 0 0"/>
         <geometry>
-          <cylinder length="0.099" radius="0.039"/>
+          <cylinder length="${($(arg hande_height) + $(arg coupler_hande_cutoff) + 0.005) / 1}" radius="0.039"/>
         </geometry>
       </collision>
       <inertial>
         <mass value="0.86387"/>
+        <!-- TODO: Parametrize intertia in terms of perpendicular axis to a solid cylinder -->
         <inertia ixx="1E-3" ixy="0.0" ixz="0.0" iyy="1E-3" iyz="0.0" izz="6E-4"/>
       </inertial>
     </link>
     <joint name="${prefix}robotiq_hande_left_finger_joint" type="prismatic">
-      <origin xyz="-0.025 0 0.0345" rpy="0 0 0"/>
+      <origin xyz="0 0 $(arg hande_height)" rpy="0 0 0"/>
       <parent link="${prefix}robotiq_hande_link"/>
       <child link="${prefix}robotiq_hande_left_finger"/>
@@ -79,5 +85,5 @@
     <link name="${prefix}robotiq_hande_left_finger">
       <visual>
-        <origin xyz="0 0 0" rpy="${pi/2} 0 ${pi/2}"/>
+        <origin xyz="0 0 0" rpy="0 0 0"/>
         <geometry>
           <mesh filename="package://robotiq_hande_description/meshes/finger.dae" scale="1.0 1.0 1.0"/>
@@ -85,5 +91,5 @@
       </visual>
       <collision>
-        <origin xyz="0 0 0" rpy="0 0 ${pi/2}"/>
+        <origin xyz="0 0 0" rpy="0 0 0"/>
         <geometry>
           <mesh filename="package://robotiq_hande_description/meshes/finger_collision.dae" scale="1.0 1.0 1.0"/>
@@ -97,5 +103,5 @@
     </link>
     <joint name="${prefix}robotiq_hande_right_finger_joint" type="prismatic">
-      <origin xyz="0.025 0 0.0345" rpy="0 0 0"/>
+      <origin xyz="0 0 $(arg hande_height)" rpy="0 0 0"/>
       <parent link="${prefix}robotiq_hande_link"/>
       <child link="${prefix}robotiq_hande_right_finger"/>
@@ -106,5 +112,5 @@
     <link name="${prefix}robotiq_hande_right_finger">
       <visual>
-        <origin xyz="0 0 0" rpy="${pi/2} 0 ${-pi/2}"/>
+        <origin xyz="0 0 0" rpy="0 0 ${pi}"/>
         <geometry>
           <mesh filename="package://robotiq_hande_description/meshes/finger.dae" scale="1.0 1.0 1.0"/>
@@ -112,5 +118,5 @@
       </visual>
       <collision>
-        <origin xyz="0 0 0" rpy="0 0 ${-pi/2}"/>
+        <origin xyz="0 0 0" rpy="0 0 ${pi}"/>
         <geometry>
           <mesh filename="package://robotiq_hande_description/meshes/finger_collision.dae" scale="1.0 1.0 1.0"/>
@@ -124,5 +130,5 @@
     </link>
     <joint name="${prefix}robotiq_hande_end_joint" type="fixed">
-      <origin xyz="0 0 0.095" rpy="0 0 0"/>
+      <origin xyz="0 0 ${$(arg hande_height) + 0.0465}" rpy="0 0 0"/>
       <parent link="${prefix}robotiq_hande_link"/>
       <child link="${prefix}robotiq_hande_end"/>
