Commit message: moved intertia mass centers

File: urdf/cylinder_inertial.xacro (robot description, xacro)
@@ -1,7 +1,8 @@
 <?xml version="1.0"?>
 <robot xmlns:xacro="http://ros.org/wiki/xacro">
-  <xacro:macro name="cylinder_inertial" params="r h m">
+  <xacro:macro name="cylinder_inertial" params="r h m *origin">
     <inertial>
       <mass value="${m}"/>
+      <xacro:insert_block name="origin"/>
       <inertia ixx="${0.0833333 * m * (3 * (r * r) + h * h)}" ixy="0.0" ixz="0.0" iyy="${0.0833333 * m * (3 * (r * r) + h * h)}" iyz="0.0" izz="${0.5 * m * (r * r)}"/>
     </inertial>

File: urdf/robotiq_hande_gripper.xacro (robot description, xacro)
@@ -48,5 +48,7 @@
         </geometry>
       </collision>
-      <xacro:cylinder_inertial r="$(arg hande_radius)" h="$(arg coupler_shell_height)" m="${coupler_mass}"/>
+      <xacro:cylinder_inertial r="$(arg hande_radius)" h="$(arg coupler_shell_height)" m="${coupler_mass}">
+        <origin xyz="0 0 ${$(arg coupler_shell_height) / 2 - $(arg coupler_parent_cutoff)}" rpy="0 0 0"/>
+      </xacro:cylinder_inertial>
     </link>
     <joint name="${prefix}robotiq_hande_base_joint" type="fixed">
@@ -68,5 +70,7 @@
         </geometry>
       </collision>
-      <xacro:cylinder_inertial r="$(arg hande_radius)" h="$(arg hande_height)" m="0.86387"/>
+      <xacro:cylinder_inertial r="$(arg hande_radius)" h="$(arg hande_height)" m="0.86387">
+        <origin xyz="0 0 ${$(arg hande_height) / 2}" rpy="0 0 0"/>
+      </xacro:cylinder_inertial>
     </link>
     <joint name="${prefix}robotiq_hande_left_finger_joint" type="prismatic">
