Commit message: unified naming for joints & links

File: urdf/robotiq_hande_gripper.xacro (robot description, xacro)
@@ -9,10 +9,10 @@
     <!--  + Height added by the coupler: 13.9mm -->
     <!--  + Reference frame: at the middle (6.95mm) -->
-    <joint name="robotiq_coupler_joint" type="fixed">
+    <joint name="robotiq_hande_coupler_joint" type="fixed">
       <origin xyz="0 0 0.00695" rpy="0 0 ${-pi/2.0}" />
       <parent link="${parent}"/>
-      <child link="${prefix}robotiq_coupler"/>
+      <child link="${prefix}robotiq_hande_coupler"/>
     </joint>
-    <link name="${prefix}robotiq_coupler">
+    <link name="${prefix}robotiq_hande_coupler">
       <inertial>
         <mass value="0.168" />
@@ -37,8 +37,8 @@
     <joint name="${prefix}robotiq_hande_base_joint" type="fixed">
       <origin rpy="0 0 0" xyz="0 0 0.055"/>
-      <parent link="${prefix}robotiq_coupler"/>
-      <child link="${prefix}hande_link"/>
+      <parent link="${prefix}robotiq_hande_coupler"/>
+      <child link="${prefix}robotiq_hande_link"/>
     </joint>
-    <link name="${prefix}hande_link">
+    <link name="${prefix}robotiq_hande_link">
       <inertial>
         <mass value="0.86387"/>
@@ -62,12 +62,12 @@
       </visual>
     </link>
-    <joint name="${prefix}hande_left_finger_joint" type="prismatic">
+    <joint name="${prefix}robotiq_hande_left_finger_joint" type="prismatic">
       <origin rpy="0 0 0" xyz="0 -0.025 0.0345"/>
-      <parent link="${prefix}hande_link"/>
-      <child link="${prefix}hande_left_finger"/>
+      <parent link="${prefix}robotiq_hande_link"/>
+      <child link="${prefix}robotiq_hande_left_finger"/>
       <axis xyz="0 1 0"/>
       <limit effort="130" lower="0" upper="0.025" velocity="0.15"/>
     </joint>
-    <link name="${prefix}hande_left_finger">
+    <link name="${prefix}robotiq_hande_left_finger">
       <inertial>
         <origin rpy="0 0 0" xyz="0 0 0"/>
@@ -93,13 +93,13 @@
       </visual>
     </link>
-    <joint name="${prefix}hande_right_finger_joint" type="prismatic">
+    <joint name="${prefix}robotiq_hande_right_finger_joint" type="prismatic">
       <origin rpy="0 0 0" xyz="0 0.025 0.0345"/>
-      <parent link="${prefix}hande_link"/>
-      <child link="${prefix}hande_right_finger"/>
+      <parent link="${prefix}robotiq_hande_link"/>
+      <child link="${prefix}robotiq_hande_right_finger"/>
       <axis xyz="0 -1 0"/>
       <limit effort="130" lower="0" upper="0.025" velocity="0.15"/>
-      <mimic joint="${prefix}hande_left_finger_joint" multiplier="1" offset="0"/>
+      <mimic joint="${prefix}robotiq_hande_left_finger_joint" multiplier="1" offset="0"/>
     </joint>
-    <link name="${prefix}hande_right_finger">
+    <link name="${prefix}robotiq_hande_right_finger">
       <inertial>
         <origin rpy="0 0 0" xyz="0 0 0"/>
@@ -127,8 +127,8 @@
     <joint name="${prefix}robotiq_hande_end_joint" type="fixed">
       <origin rpy="0 0 0" xyz="0 0 0.095"/>
-      <parent link="${prefix}hande_link"/>
-      <child link="${prefix}hande_end"/>
+      <parent link="${prefix}robotiq_hande_link"/>
+      <child link="${prefix}robotiq_hande_end"/>
     </joint>
-    <link name="${prefix}hande_end" />
+    <link name="${prefix}robotiq_hande_end" />
   </xacro:macro>
 </robot>

Commit message: improved urdf readability

File: urdf/robotiq_hande_gripper.xacro (robot description, xacro)
@@ -18,13 +18,4 @@
     </joint>
     <link name="${prefix}robotiq_hande_coupler">
-      <inertial>
-        <mass value="0.168"/>
-        <inertia ixx="6.17674E-05" ixy="0.0" ixz="0.0" iyy="6.17674E-05" iyz="0.0" izz="1.18125E-04"/>
-      </inertial>
-      <collision>
-        <geometry>
-          <cylinder length="0.0139" radius="0.0375"/>
-        </geometry>
-      </collision>
       <visual>
         <geometry>
@@ -33,15 +24,27 @@
         <material name="DarkGrey"/>
       </visual>
+      <collision>
+        <geometry>
+          <cylinder length="0.0139" radius="0.0375"/>
+        </geometry>
+      </collision>
+      <inertial>
+        <mass value="0.168"/>
+        <inertia ixx="6.17674E-05" ixy="0.0" ixz="0.0" iyy="6.17674E-05" iyz="0.0" izz="1.18125E-04"/>
+      </inertial>
     </link>
     <joint name="${prefix}robotiq_hande_base_joint" type="fixed">
-      <origin rpy="0 0 0" xyz="0 0 0.055"/>
+      <origin xyz="0 0 0.055" rpy="0 0 0"/>
       <parent link="${prefix}robotiq_hande_coupler"/>
       <child link="${prefix}robotiq_hande_link"/>
     </joint>
     <link name="${prefix}robotiq_hande_link">
-      <inertial>
-        <mass value="0.86387"/>
-        <inertia ixx="0.001" ixy="0.0" ixz="0.0" iyy="0.001" iyz="0.0" izz="0.0006"/>
-      </inertial>
+      <visual>
+        <origin xyz="0 0 -0.0016" rpy="0 ${-pi/2} ${-pi/2}"/>
+        <geometry>
+          <mesh filename="package://robotiq_hande_description/meshes/hande.dae" scale="1.0 1.0 1.0"/>
+        </geometry>
+        <material name="DarkGrey"/>
+      </visual>
       <collision>
         <geometry>
@@ -49,14 +52,11 @@
         </geometry>
       </collision>
-      <visual>
-        <origin rpy="0 -1.570796 -1.570796" xyz="0 0 -0.0016"/>
-        <geometry>
-          <mesh filename="package://robotiq_hande_description/meshes/hande.dae" scale="1.0 1.0 1.0"/>
-        </geometry>
-        <material name="DarkGrey"/>
-      </visual>
+      <inertial>
+        <mass value="0.86387"/>
+        <inertia ixx="0.001" ixy="0.0" ixz="0.0" iyy="0.001" iyz="0.0" izz="0.0006"/>
+      </inertial>
     </link>
     <joint name="${prefix}robotiq_hande_left_finger_joint" type="prismatic">
-      <origin rpy="0 0 0" xyz="0 -0.025 0.0345"/>
+      <origin xyz="0 -0.025 0.0345" rpy="0 0 0"/>
       <parent link="${prefix}robotiq_hande_link"/>
       <child link="${prefix}robotiq_hande_left_finger"/>
@@ -65,17 +65,6 @@
     </joint>
     <link name="${prefix}robotiq_hande_left_finger">
-      <inertial>
-        <origin rpy="0 0 0" xyz="0 0 0"/>
-        <mass value="0.03804"/>
-        <inertia ixx="1E-9" ixy="0.0" ixz="0.0" iyy="1E-9" iyz="0.0" izz="1E-9"/>
-      </inertial>
-      <collision>
-        <origin rpy="0 0 3.1415926" xyz="0 0 0"/>
-        <geometry>
-          <mesh filename="package://robotiq_hande_description/meshes/finger_collision.dae" scale="1.0 1.0 1.0"/>
-        </geometry>
-      </collision>
       <visual>
-        <origin rpy="1.570796 0 3.1415926" xyz="0 0 0"/>
+        <origin xyz="0 0 0" rpy="${pi/2} 0 ${pi}"/>
         <geometry>
           <mesh filename="package://robotiq_hande_description/meshes/finger.dae" scale="1.0 1.0 1.0"/>
@@ -83,7 +72,18 @@
         <material name="Grey"/>
       </visual>
+      <collision>
+        <origin xyz="0 0 0" rpy="0 0 ${pi}"/>
+        <geometry>
+          <mesh filename="package://robotiq_hande_description/meshes/finger_collision.dae" scale="1.0 1.0 1.0"/>
+        </geometry>
+      </collision>
+      <inertial>
+        <origin xyz="0 0 0" rpy="0 0 0"/>
+        <mass value="0.03804"/>
+        <inertia ixx="1E-9" ixy="0.0" ixz="0.0" iyy="1E-9" iyz="0.0" izz="1E-9"/>
+      </inertial>
     </link>
     <joint name="${prefix}robotiq_hande_right_finger_joint" type="prismatic">
-      <origin rpy="0 0 0" xyz="0 0.025 0.0345"/>
+      <origin xyz="0 0.025 0.0345" rpy="0 0 0"/>
       <parent link="${prefix}robotiq_hande_link"/>
       <child link="${prefix}robotiq_hande_right_finger"/>
@@ -93,17 +93,6 @@
     </joint>
     <link name="${prefix}robotiq_hande_right_finger">
-      <inertial>
-        <origin rpy="0 0 0" xyz="0 0 0"/>
-        <mass value="0.03804"/>
-        <inertia ixx="1E-9" ixy="0.0" ixz="0.0" iyy="1E-9" iyz="0.0" izz="1E-9"/>
-      </inertial>
-      <collision>
-        <origin rpy="0 0 0" xyz="0 0 0"/>
-        <geometry>
-          <mesh filename="package://robotiq_hande_description/meshes/finger_collision.dae" scale="1.0 1.0 1.0"/>
-        </geometry>
-      </collision>
       <visual>
-        <origin rpy="1.570796 0 0" xyz="0 0 0"/>
+        <origin xyz="0 0 0" rpy="${pi/2} 0 0"/>
         <geometry>
           <mesh filename="package://robotiq_hande_description/meshes/finger.dae" scale="1.0 1.0 1.0"/>
@@ -111,7 +100,18 @@
         <material name="Grey"/>
       </visual>
+      <collision>
+        <origin xyz="0 0 0" rpy="0 0 0"/>
+        <geometry>
+          <mesh filename="package://robotiq_hande_description/meshes/finger_collision.dae" scale="1.0 1.0 1.0"/>
+        </geometry>
+      </collision>
+      <inertial>
+        <origin xyz="0 0 0" rpy="0 0 0"/>
+        <mass value="0.03804"/>
+        <inertia ixx="1E-9" ixy="0.0" ixz="0.0" iyy="1E-9" iyz="0.0" izz="1E-9"/>
+      </inertial>
     </link>
     <joint name="${prefix}robotiq_hande_end_joint" type="fixed">
-      <origin rpy="0 0 0" xyz="0 0 0.095"/>
+      <origin xyz="0 0 0.095" rpy="0 0 0"/>
       <parent link="${prefix}robotiq_hande_link"/>
       <child link="${prefix}robotiq_hande_end"/>

Commit message: removed unused materials colours (for dae files)

File: urdf/robotiq_hande_gripper.xacro (robot description, xacro)
@@ -22,5 +22,4 @@
           <mesh filename="package://robotiq_hande_description/meshes/coupler.dae"/>
         </geometry>
-        <material name="DarkGrey"/>
       </visual>
       <collision>
@@ -45,5 +44,4 @@
           <mesh filename="package://robotiq_hande_description/meshes/hande.dae" scale="1.0 1.0 1.0"/>
         </geometry>
-        <material name="DarkGrey"/>
       </visual>
       <collision>
@@ -70,5 +68,4 @@
           <mesh filename="package://robotiq_hande_description/meshes/finger.dae" scale="1.0 1.0 1.0"/>
         </geometry>
-        <material name="Grey"/>
       </visual>
       <collision>
@@ -98,5 +95,4 @@
           <mesh filename="package://robotiq_hande_description/meshes/finger.dae" scale="1.0 1.0 1.0"/>
         </geometry>
-        <material name="Grey"/>
       </visual>
       <collision>

Commit message: unified inertial notation

File: urdf/robotiq_hande_gripper.xacro (robot description, xacro)
@@ -30,5 +30,5 @@
       <inertial>
         <mass value="0.168"/>
-        <inertia ixx="6.17674E-05" ixy="0.0" ixz="0.0" iyy="6.17674E-05" iyz="0.0" izz="1.18125E-04"/>
+        <inertia ixx="6.17674E-5" ixy="0.0" ixz="0.0" iyy="6.17674E-5" iyz="0.0" izz="1.18125E-4"/>
       </inertial>
     </link>
@@ -52,5 +52,5 @@
       <inertial>
         <mass value="0.86387"/>
-        <inertia ixx="0.001" ixy="0.0" ixz="0.0" iyy="0.001" iyz="0.0" izz="0.0006"/>
+        <inertia ixx="1E-3" ixy="0.0" ixz="0.0" iyy="1E-3" iyz="0.0" izz="6E-4"/>
       </inertial>
     </link>

Commit message: parametrized coupler mass (with bolts)

File: urdf/robotiq_hande_gripper.xacro (robot description, xacro)
@@ -6,5 +6,5 @@
   <xacro:include filename="$(find robotiq_hande_description)/urdf/materials.xacro"/>
   <xacro:include filename="$(find robotiq_hande_description)/urdf/robotiq_hande_gripper.ros2_control.xacro"/>
-  <xacro:macro name="robotiq_hande_gripper" params="name prefix parent tty use_fake_hardware">
+  <xacro:macro name="robotiq_hande_gripper" params="name prefix parent tty use_fake_hardware coupler_mass:=0.119">
     <!-- ros2_control parameters  -->
     <xacro:robotiq_hande_ros2_control name="${name}" prefix="${prefix}" tty="${tty}" use_fake_hardware="${use_fake_hardware}"/>
@@ -12,4 +12,5 @@
     <!--  + Height added by the coupler (13.9mm) -->
     <!--  + Reference frame at the middle (6.95mm) -->
+    <!--  + Mass includes the bolts -->
     <joint name="${prefix}robotiq_hande_coupler_joint" type="fixed">
       <origin xyz="0 0 0.00695" rpy="0 0 ${-pi/2.0}"/>
@@ -29,5 +30,5 @@
       </collision>
       <inertial>
-        <mass value="0.168"/>
+        <mass value="${coupler_mass}"/>
         <inertia ixx="6.17674E-5" ixy="0.0" ixz="0.0" iyy="6.17674E-5" iyz="0.0" izz="1.18125E-4"/>
       </inertial>

Commit message: updated models (new io coupler)

File: urdf/robotiq_hande_gripper.xacro (robot description, xacro)
@@ -4,5 +4,4 @@
     Based on the URDF file by Cristian C Beltran-Hernandez
   -->
-  <xacro:include filename="$(find robotiq_hande_description)/urdf/materials.xacro"/>
   <xacro:include filename="$(find robotiq_hande_description)/urdf/robotiq_hande_gripper.ros2_control.xacro"/>
   <xacro:macro name="robotiq_hande_gripper" params="name prefix parent tty use_fake_hardware coupler_mass:=0.119">
@@ -10,7 +9,10 @@
     <xacro:robotiq_hande_ros2_control name="${name}" prefix="${prefix}" tty="${tty}" use_fake_hardware="${use_fake_hardware}"/>
     <!-- Robotiq Coupler -->
-    <!--  + Height added by the coupler (13.9mm) -->
+    <!--  + Height added by the coupler (16.9mm) -->
     <!--  + Reference frame at the middle (6.95mm) -->
-    <!--  + Mass includes the bolts -->
+    <!--  + Coupler mass includes the bolts -->
+    <xacro:arg name="base_joint_z_offset" default="0.055"/>
+    <xacro:arg name="coupler_depth" default="0.00294"/>
+    <xacro:arg name="base_to_coupler_offset" default="0.00145"/>
     <joint name="${prefix}robotiq_hande_coupler_joint" type="fixed">
       <origin xyz="0 0 0.00695" rpy="0 0 ${-pi/2.0}"/>
@@ -21,10 +23,10 @@
       <visual>
         <geometry>
-          <mesh filename="package://robotiq_hande_description/meshes/coupler.dae"/>
+          <mesh filename="package://robotiq_hande_description/meshes/io_coupler.dae"/>
         </geometry>
       </visual>
       <collision>
         <geometry>
-          <cylinder length="0.0139" radius="0.0375"/>
+          <cylinder length="0.014" radius="0.039"/>
         </geometry>
       </collision>
@@ -35,5 +37,5 @@
     </link>
     <joint name="${prefix}robotiq_hande_base_joint" type="fixed">
-      <origin xyz="0 0 0.055" rpy="0 0 0"/>
+      <origin xyz="0 0 ${$(arg base_joint_z_offset) + $(arg coupler_depth) - $(arg base_to_coupler_offset)}" rpy="0 0 0"/>
       <parent link="${prefix}robotiq_hande_coupler"/>
       <child link="${prefix}robotiq_hande_link"/>
@@ -41,5 +43,5 @@
     <link name="${prefix}robotiq_hande_link">
       <visual>
-        <origin xyz="0 0 -0.0016" rpy="0 ${-pi/2} ${-pi/2}"/>
+        <origin xyz="0 0 0" rpy="0 ${-pi/2} 0"/>
         <geometry>
           <mesh filename="package://robotiq_hande_description/meshes/hande.dae" scale="1.0 1.0 1.0"/>
@@ -48,5 +50,5 @@
       <collision>
         <geometry>
-          <cylinder length="0.0988" radius="0.0375"/>
+          <cylinder length="0.099" radius="0.039"/>
         </geometry>
       </collision>
@@ -57,13 +59,13 @@
     </link>
     <joint name="${prefix}robotiq_hande_left_finger_joint" type="prismatic">
-      <origin xyz="0 -0.025 0.0345" rpy="0 0 0"/>
+      <origin xyz="-0.025 0 0.0345" rpy="0 0 0"/>
       <parent link="${prefix}robotiq_hande_link"/>
       <child link="${prefix}robotiq_hande_left_finger"/>
-      <axis xyz="0 1 0"/>
+      <axis xyz="1 0 0"/>
       <limit effort="130" lower="0" upper="0.025" velocity="0.15"/>
     </joint>
     <link name="${prefix}robotiq_hande_left_finger">
       <visual>
-        <origin xyz="0 0 0" rpy="${pi/2} 0 ${pi}"/>
+        <origin xyz="0 0 0" rpy="${pi/2} 0 ${pi/2}"/>
         <geometry>
           <mesh filename="package://robotiq_hande_description/meshes/finger.dae" scale="1.0 1.0 1.0"/>
@@ -71,5 +73,5 @@
       </visual>
       <collision>
-        <origin xyz="0 0 0" rpy="0 0 ${pi}"/>
+        <origin xyz="0 0 0" rpy="0 0 ${pi/2}"/>
         <geometry>
           <mesh filename="package://robotiq_hande_description/meshes/finger_collision.dae" scale="1.0 1.0 1.0"/>
@@ -83,8 +85,8 @@
     </link>
     <joint name="${prefix}robotiq_hande_right_finger_joint" type="prismatic">
-      <origin xyz="0 0.025 0.0345" rpy="0 0 0"/>
+      <origin xyz="0.025 0 0.0345" rpy="0 0 0"/>
       <parent link="${prefix}robotiq_hande_link"/>
       <child link="${prefix}robotiq_hande_right_finger"/>
-      <axis xyz="0 -1 0"/>
+      <axis xyz="-1 0 0"/>
       <limit effort="130" lower="0" upper="0.025" velocity="0.15"/>
       <mimic joint="${prefix}robotiq_hande_left_finger_joint" multiplier="1" offset="0"/>
@@ -92,5 +94,5 @@
     <link name="${prefix}robotiq_hande_right_finger">
       <visual>
-        <origin xyz="0 0 0" rpy="${pi/2} 0 0"/>
+        <origin xyz="0 0 0" rpy="${pi/2} 0 ${-pi/2}"/>
         <geometry>
           <mesh filename="package://robotiq_hande_description/meshes/finger.dae" scale="1.0 1.0 1.0"/>
@@ -98,5 +100,5 @@
       </visual>
       <collision>
-        <origin xyz="0 0 0" rpy="0 0 0"/>
+        <origin xyz="0 0 0" rpy="0 0 ${-pi/2}"/>
         <geometry>
           <mesh filename="package://robotiq_hande_description/meshes/finger_collision.dae" scale="1.0 1.0 1.0"/>

Commit message: Added cylinder inertial

File: urdf/robotiq_hande_gripper.xacro (robot description, xacro)
@@ -5,4 +5,5 @@
   -->
   <xacro:include filename="$(find robotiq_hande_description)/urdf/robotiq_hande_gripper.ros2_control.xacro"/>
+  <xacro:include filename="$(find robotiq_hande_description)/urdf/cylinder_inertial.xacro"/>
   <xacro:macro name="robotiq_hande_gripper" params="name prefix parent grip_pos_min grip_pos_max tty baudrate parity data_bits stop_bit slave_id use_fake_hardware coupler_mass:=0.119">
     <!-- ros2_control parameters  -->
@@ -29,4 +30,5 @@
     <xacro:arg name="coupler_hande_cutoff" default="0.0029"/>
     <xacro:arg name="hande_height" default="0.099"/>
+    <xacro:arg name="hande_radius" default="0.0375"/>
     <joint name="${prefix}robotiq_hande_coupler_joint" type="fixed">
       <origin xyz="0 0 0" rpy="0 0 ${-pi/2.0}"/>
@@ -46,9 +48,5 @@
         </geometry>
       </collision>
-      <inertial>
-        <mass value="${coupler_mass}"/>
-        <!-- TODO: Parametrize inertia in terms of perpendicular axis to a solid cylinder -->
-        <inertia ixx="6.17674E-5" ixy="0.0" ixz="0.0" iyy="6.17674E-5" iyz="0.0" izz="1.18125E-4"/>
-      </inertial>
+      <xacro:cylinder_inertial r="$(arg hande_radius)" h="$(arg coupler_shell_height)" m="${coupler_mass}"/>
     </link>
     <joint name="${prefix}robotiq_hande_base_joint" type="fixed">
@@ -70,9 +68,5 @@
         </geometry>
       </collision>
-      <inertial>
-        <mass value="0.86387"/>
-        <!-- TODO: Parametrize inertia in terms of perpendicular axis to a solid cylinder -->
-        <inertia ixx="1E-3" ixy="0.0" ixz="0.0" iyy="1E-3" iyz="0.0" izz="6E-4"/>
-      </inertial>
+      <xacro:cylinder_inertial r="$(arg hande_radius)" h="$(arg hande_height)" m="0.86387"/>
     </link>
     <joint name="${prefix}robotiq_hande_left_finger_joint" type="prismatic">

Commit message: parametrized collision cylinders with hande_radius

File: urdf/robotiq_hande_gripper.xacro (robot description, xacro)
@@ -2,5 +2,5 @@
 <robot xmlns:xacro="http://ros.org/wiki/xacro">
   <!--
-    Based on the URDF file by Cristian C Beltran-Hernandez
+    Original URDF file by Cristian C Beltran-Hernandez
   -->
   <xacro:include filename="$(find robotiq_hande_description)/urdf/robotiq_hande_gripper.ros2_control.xacro"/>
@@ -45,5 +45,5 @@
         <origin xyz="0 0 ${$(arg coupler_shell_height)/2 - $(arg coupler_parent_cutoff)}" rpy="0 0 0"/>
         <geometry>
-          <cylinder length="$(arg coupler_shell_height)" radius="0.039"/>
+          <cylinder length="$(arg coupler_shell_height)" radius="${$(arg hande_radius) + 0.001}"/>
         </geometry>
       </collision>
@@ -65,5 +65,5 @@
         <origin xyz="0 0 ${($(arg hande_height) + $(arg coupler_hande_cutoff) + 0.005) / 2}" rpy="0 0 0"/>
         <geometry>
-          <cylinder length="${($(arg hande_height) + $(arg coupler_hande_cutoff) + 0.005) / 1}" radius="0.039"/>
+          <cylinder length="${$(arg hande_height) + $(arg coupler_hande_cutoff) + 0.005}" radius="${$(arg hande_radius) + 0.001}"/>
         </geometry>
       </collision>

Commit message: fixed default rotatation of hande

File: urdf/robotiq_hande_gripper.xacro (robot description, xacro)
@@ -32,5 +32,5 @@
     <xacro:arg name="hande_radius" default="0.0375"/>
     <joint name="${prefix}robotiq_hande_coupler_joint" type="fixed">
-      <origin xyz="0 0 0" rpy="0 0 ${-pi/2.0}"/>
+      <origin xyz="0 0 0" rpy="0 0 0"/>
       <parent link="${parent}"/>
       <child link="${prefix}robotiq_hande_coupler"/>

Commit message: Make gripper mounting pose configurable

File: urdf/robotiq_hande_gripper.xacro (robot description, xacro)
@@ -6,5 +6,21 @@
   <xacro:include filename="$(find robotiq_hande_description)/urdf/robotiq_hande_gripper.ros2_control.xacro"/>
   <xacro:include filename="$(find robotiq_hande_description)/urdf/cylinder_inertial.xacro"/>
-  <xacro:macro name="robotiq_hande_gripper" params="name prefix parent grip_pos_min grip_pos_max tty baudrate parity data_bits stop_bit slave_id use_fake_hardware coupler_mass:=0.119">
+  <xacro:macro
+    name="robotiq_hande_gripper"
+    params="name
+            prefix
+            parent
+            grip_pos_min
+            grip_pos_max
+            tty
+            baudrate
+            parity
+            data_bits
+            stop_bit
+            slave_id
+            use_fake_hardware
+            coupler_mass:=0.119
+            xyz:='0 0 0'
+            rpy:='0 0 0'">
     <!-- ros2_control parameters  -->
     <xacro:robotiq_hande_ros2_control
@@ -32,5 +48,5 @@
     <xacro:arg name="hande_radius" default="0.0375"/>
     <joint name="${prefix}robotiq_hande_coupler_joint" type="fixed">
-      <origin xyz="0 0 0" rpy="0 0 0"/>
+      <origin xyz="${xyz}" rpy="${rpy}"/>
       <parent link="${parent}"/>
       <child link="${prefix}robotiq_hande_coupler"/>
